Commit message: perceptive locomotion demo initial test passed

File: ocs2_robotic_examples/ocs2_perceptive_anymal/ocs2_anymal_models/urdf/anymal_camel_rsl.urdf (robot description, URDF)
Before this commit: robot anymal, 69 links, 68 joints
Links:
- link base: geometry collision box size=0.58 0.14 0.18; collision cylinder length=0.145 radius=0.09
